Commit message: correcting merge conflicts on urdf file

File: my_rb1_description/urdf/my_rb1_robot.urdf (robot description, URDF)
Before this commit: robot rb1_robot, 7 links, 6 joints
Links:
- link front_laser: mass 0.5 -> None; geometry 
Joints:
- joint base_link_back_caster_joint: axis (none) -> 0 0 1; type fixed -> continuous
- joint base_link_front_caster_joint: axis (none) -> 0 0 1; type fixed -> continuous
- joint base_link_front_laser_joint: origin xyz=0.8 0 0.3 rpy=0 0 0 -> xyz=0.25 0.0 0.075 rpy=3.14159265 0 0

Commit message: Added properties to front-laser link & positioned it rightly

File: my_rb1_description/urdf/my_rb1_robot.urdf (robot description, URDF)
Before this commit: robot rb1_robot, 7 links, 6 joints
Links:
- link front_laser: mass None -> 0.1; geometry collision cylinder length=0.1 radius=0.05; visual cylinder length=0.1 radius=0.05
Joints:
- joint joint_laser_scan_chassis: origin xyz=0.8 0 0.3 rpy=0 0 0 -> xyz=0.25 0 0.3 rpy=0 0 0

Commit message: Changed color of the gazebo model

File: my_rb1_description/urdf/my_rb1_robot.urdf (robot description, URDF)
Before this commit: robot rb1_robot, 7 links, 6 joints
Links:
- link front_laser: mass 0.5 -> 0.1
Joints:
- joint base_link_front_laser_joint: origin xyz=0.8 0 0.3 rpy=0 0 0 -> xyz=0.25 0 0.15 rpy=0 0 0

Commit message: Got the robot moving

File: my_rb1_description/urdf/my_rb1_robot.urdf (robot description, URDF)
Before this commit: robot rb1_robot, 7 links, 6 joints
Links:
- link back_caster: mass 0.2 -> 0.1
- link front_caster: mass 0.2 -> 0.1
- link front_laser: mass None -> 0.01; geometry visual cylinder length=0.01 radius=0.01
Joints:
- removed joint base_link_back_caster_joint
- removed joint base_link_front_caster_joint
- removed joint base_link_front_laser_joint
- removed joint base_link_plate_joint
- added joint back_caster_joint: type fixed, parent base_link, child back_caster, origin xyz=-0.1 0.0 -0.15
- added joint base_link_joint: type fixed, parent base_footprint, child base_link, origin xyz=0 0 0.15 rpy=0 0 0
- added joint front_caster_joint: type fixed, parent base_link, child front_caster, origin xyz=0.1 0.0 -0.15
- added joint front_laser_joint: type fixed, parent base_link, child front_laser, origin xyz=0.25 0.0 0.075 rpy=0 0 0
